Commit message: Working line follower robot with custom world and proportional ang_vel adjustment

File: install/my_robot_description/share/my_robot_description/urdf/camera.urdf.xacro (robot description, xacro)
@@ -24,5 +24,5 @@
         <parent link = "base_link" />
         <child link = "camera_link" />
-        <origin xyz = "${(base_length+camera_length)/2.0} 0 ${base_height/2.0}" rpy = "0 0 0" />
+        <origin xyz = "${(base_length+camera_length)/2.0} 0 ${base_height}" rpy = "0 ${pi/3.0} 0" />
     </joint>
     <link name="camera_link_optical"/>
